File: MotorBoard_v7/MotorBoard.kicad_sch (KiCad schematic)
At the start: 4 parts

Commit message: lab5 done
Other:
- note added: "3.3V_ESP"
- note added: "Each LM2937 can supply 400mA of 3.3V"
- note added: "Motor Board: 3.3V_ESP ESP 3.3V SSD1306 VOUT 5.0V Servo (not powered) 11.1 DC motors (not powered)"
- note added: "Motor Board: 3.3V_ESP ESP 3.3V SSD1306 VOUT 5.0V Servo 11.1 DC motors"
- note removed: "LM2937 can supply 400mA of 3.3V"
- note removed: "Motor Board: 3.3V SSD1306 ESP VOUT 5.0V Servo (not powered) 11.1 DC motors (not powered)"
- note removed: "Motor Board: 3.3V SSD1306 ESP VOUT 5.0V Servo 11.1 DC motors"
